Commit message: checking changes

File: src/hexapod_ws/description/hexapod.urdf.xacro (robot description, xacro)
@@ -1,8 +1,4 @@
 <?xml version="1.0"?>
 <robot xmlns:xacro="http://www.ros.org/wiki/xacro" name="hexapod">
-  <xacro:include filename="$(find hexapod_ws)/description/hexapod.gazebo"/>
-  <xacro:property name="name_prefix" value=""/>
-  <xacro:property name="joint_lower_limit" value="-1.57"/>
-  <xacro:property name="joint_upper_limit" value="1.57"/>
   <xacro:property name="base_radius" value="0.18"/>
   <xacro:property name="base_height" value="0.05"/>
@@ -11,173 +7,234 @@
   <xacro:property name="tibia_length" value="0.18"/>
   <xacro:property name="leg_radius" value="0.01"/>
-  <link name="base_footprint"/>
-  <joint name="base_joint" type="fixed">
-    <parent link="base_footprint"/>
-    <child link="base_link"/>
-    <origin xyz="0 0 0" rpy="0 0 0"/>
-  </joint>
+  <xacro:property name="joint_lower_limit" value="-1.57"/>
+  <xacro:property name="joint_upper_limit" value="1.57"/>
+  <!-- Base Link -->
   <link name="base_link">
     <inertial>
       <origin xyz="0 0 0" rpy="0 0 0"/>
-      <mass value="2.5"/>
-      <inertia ixx="0.02077" ixy="0.0" ixz="0.0" iyy="0.02077" iyz="0.0" izz="0.0405"/>
+      <mass value="3.0"/>
+      <inertia ixx="0.02" ixy="0.0" ixz="0.0" iyy="0.02" iyz="0.0" izz="0.02"/>
     </inertial>
     <visual>
       <origin xyz="0 0 ${base_height/2}" rpy="0 0 0"/>
-      <geometry><cylinder radius="${base_radius}" length="${base_height}"/></geometry>
-      <material name="gray"><color rgba="0.6 0.6 0.6 1.0"/></material>
+      <geometry>
+        <cylinder radius="${base_radius}" length="${base_height}"/>
+      </geometry>
+      <material name="gray">
+        <color rgba="0.6 0.6 0.6 1.0"/>
+      </material>
     </visual>
     <collision>
       <origin xyz="0 0 ${base_height/2}" rpy="0 0 0"/>
-      <geometry><cylinder radius="${base_radius}" length="${base_height}"/></geometry>
+      <geometry>
+        <cylinder radius="${base_radius}" length="${base_height}"/>
+      </geometry>
     </collision>
   </link>
+  <!-- IMU Sensor -->
   <link name="imu_link">
-    <visual>
-      <geometry><box size="0.02 0.02 0.02"/></geometry>
-      <material name="white"><color rgba="1 1 1 1"/></material>
-    </visual>
     <inertial>
-      <origin xyz="0 0 0" rpy="0 0 0"/>
-      <mass value="0.005"/>
-      <inertia ixx="2.08e-07" ixy="0" ixz="0" iyy="2.08e-07" iyz="0" izz="3.33e-07"/>
+      <mass value="0.001"/>
+      <inertia ixx="1e-6" ixy="0" ixz="0" iyy="1e-6" iyz="0" izz="1e-6"/>
     </inertial>
   </link>
   <joint name="imu_joint" type="fixed">
-    <origin xyz="0 0 ${base_height+0.02}" rpy="0 0 0"/>
+    <origin xyz="0 0 0.07" rpy="0 0 0"/>
     <parent link="base_link"/>
     <child link="imu_link"/>
   </joint>
+  <!-- LiDAR Sensor -->
   <link name="lidar_link">
+    <inertial>
+      <mass value="0.05"/>
+      <inertia ixx="1e-4" ixy="0" ixz="0" iyy="1e-4" iyz="0" izz="1e-4"/>
+    </inertial>
     <visual>
-      <geometry><cylinder radius="0.04" length="0.05"/></geometry>
-      <material name="black"><color rgba="0.1 0.1 0.1 1.0"/></material>
+      <origin xyz="0 0 0" rpy="0 0 0"/>
+      <geometry>
+        <cylinder radius="0.04" length="0.05"/>
+      </geometry>
+      <material name="black">
+        <color rgba="0.1 0.1 0.1 1.0"/>
+      </material>
     </visual>
     <collision>
-      <geometry><cylinder radius="0.04" length="0.05"/></geometry>
+      <origin xyz="0 0 0" rpy="0 0 0"/>
+      <geometry>
+        <cylinder radius="0.04" length="0.05"/>
+      </geometry>
     </collision>
-    <inertial>
-      <mass value="0.1"/>
-      <inertia ixx="1e-4" ixy="0" ixz="0" iyy="1e-4" iyz="0" izz="1e-4"/>
-    </inertial>
   </link>
   <joint name="lidar_joint" type="fixed">
-    <origin xyz="0 0 ${base_height+0.05}" rpy="0 0 0"/>
+    <origin xyz="0 0 0.1" rpy="0 0 0"/>
     <parent link="base_link"/>
     <child link="lidar_link"/>
   </joint>
   <!-- LEG MACRO -->
-  <xacro:macro name="leg" params="leg_name hx hy hz hr hp hyaw">
-    <!-- Hip Link -->
+  <xacro:macro name="leg" params="leg_name hx hy angle">
+    <!-- Hip Link (Coxa) -->
     <link name="${leg_name}_hip_link">
-      <visual>
-        <geometry><cylinder radius="${leg_radius}" length="${hip_length}"/></geometry>
-        <material name="blue"><color rgba="0 0 1 1"/></material>
+      <inertial>
+        <origin xyz="${hip_length/2} 0 0" rpy="0 1.5708 0"/>
+        <mass value="0.05"/>
+        <inertia ixx="1e-4" ixy="0" ixz="0" iyy="1e-4" iyz="0" izz="1e-4"/>
+      </inertial>
+      <visual>
+        <origin xyz="${hip_length/2} 0 0" rpy="0 1.5708 0"/>
+        <geometry>
+          <cylinder radius="${leg_radius}" length="${hip_length}"/>
+        </geometry>
+        <material name="black">
+          <color rgba="0.1 0.1 0.1 1.0"/>
+        </material>
       </visual>
       <collision>
-        <geometry><cylinder radius="${leg_radius}" length="${hip_length}"/></geometry>
-      </collision>
-      <inertial>
-        <mass value="0.1"/>
-        <inertia ixx="2.08e-05" ixy="0" ixz="0" iyy="2.08e-05" iyz="0" izz="5e-07"/>
-      </inertial>
+        <origin xyz="${hip_length/2} 0 0" rpy="0 1.5708 0"/>
+        <geometry>
+          <cylinder radius="${leg_radius}" length="${hip_length}"/>
+        </geometry>
+      </collision>
     </link>
     <joint name="${leg_name}_hip_joint" type="revolute">
+      <origin xyz="${hx} ${hy} ${base_height/2}" rpy="0 0 ${angle}"/>
       <parent link="base_link"/>
       <child link="${leg_name}_hip_link"/>
-      <origin xyz="${hx} ${hy} ${hz}" rpy="${hr} ${hp} ${hyaw}"/>
       <axis xyz="0 0 1"/>
-      <limit lower="${joint_lower_limit}" upper="${joint_upper_limit}" effort="10" velocity="1.0"/>
+      <limit lower="${joint_lower_limit}" upper="${joint_upper_limit}" effort="10" velocity="4"/>
     </joint>
     <!-- Femur Link -->
     <link name="${leg_name}_femur_link">
-      <visual>
-        <origin xyz="0 0 ${-femur_length/2}" rpy="0 0 0"/>
-        <geometry><cylinder radius="${leg_radius}" length="${femur_length}"/></geometry>
-        <material name="green"><color rgba="0 1 0 1"/></material>
+      <inertial>
+        <origin xyz="${femur_length/2} 0 0" rpy="0 1.5708 0"/>
+        <mass value="0.08"/>
+        <inertia ixx="1e-4" ixy="0" ixz="0" iyy="1e-4" iyz="0" izz="1e-4"/>
+      </inertial>
+      <visual>
+        <origin xyz="${femur_length/2} 0 0" rpy="0 1.5708 0"/>
+        <geometry>
+          <cylinder radius="${leg_radius}" length="${femur_length}"/>
+        </geometry>
+        <material name="red">
+          <color rgba="0.8 0.2 0.2 1.0"/>
+        </material>
       </visual>
       <collision>
-        <origin xyz="0 0 ${-femur_length/2}" rpy="0 0 0"/>
-        <geometry><cylinder radius="${leg_radius}" length="${femur_length}"/></geometry>
-      </collision>
-      <inertial>
-        <origin xyz="0 0 ${-femur_length/2}" rpy="0 0 0"/>
-        <mass value="0.15"/>
-        <inertia ixx="1.8e-04" ixy="0" ixz="0" iyy="1.8e-04" iyz="0" izz="1.125e-06"/>
-      </inertial>
+        <origin xyz="${femur_length/2} 0 0" rpy="0 1.5708 0"/>
+        <geometry>
+          <cylinder radius="${leg_radius}" length="${femur_length}"/>
+        </geometry>
+      </collision>
     </link>
     <joint name="${leg_name}_femur_joint" type="revolute">
+      <origin xyz="${hip_length} 0 0" rpy="0 0 0"/>
       <parent link="${leg_name}_hip_link"/>
       <child link="${leg_name}_femur_link"/>
-      <origin xyz="0 0 0" rpy="0 0 0"/>
       <axis xyz="0 1 0"/>
-      <limit lower="${joint_lower_limit}" upper="${joint_upper_limit}" effort="10" velocity="1.0"/>
+      <limit lower="${joint_lower_limit}" upper="${joint_upper_limit}" effort="10" velocity="4"/>
     </joint>
     <!-- Tibia Link -->
     <link name="${leg_name}_tibia_link">
-      <visual>
-        <origin xyz="0 0 ${-tibia_length/2}" rpy="0 0 0"/>
-        <geometry><cylinder radius="${leg_radius}" length="${tibia_length}"/></geometry>
-        <material name="red"><color rgba="1 0 0 1"/></material>
+      <inertial>
+        <origin xyz="${tibia_length/2} 0 0" rpy="0 1.5708 0"/>
+        <mass value="0.06"/>
+        <inertia ixx="1e-4" ixy="0" ixz="0" iyy="1e-4" iyz="0" izz="1e-4"/>
+      </inertial>
+      <visual>
+        <origin xyz="${tibia_length/2} 0 0" rpy="0 1.5708 0"/>
+        <geometry>
+          <cylinder radius="${leg_radius}" length="${tibia_length}"/>
+        </geometry>
+        <material name="blue">
+          <color rgba="0.2 0.2 0.8 1.0"/>
+        </material>
       </visual>
       <collision>
-        <origin xyz="0 0 ${-tibia_length/2}" rpy="0 0 0"/>
-        <geometry><cylinder radius="${leg_radius}" length="${tibia_length}"/></geometry>
-      </collision>
-      <inertial>
-        <origin xyz="0 0 ${-tibia_length/2}" rpy="0 0 0"/>
-        <mass value="0.12"/>
-        <inertia ixx="3.24e-04" ixy="0" ixz="0" iyy="3.24e-04" iyz="0" izz="7.2e-07"/>
-      </inertial>
+        <origin xyz="${tibia_length/2} 0 0" rpy="0 1.5708 0"/>
+        <geometry>
+          <cylinder radius="${leg_radius}" length="${tibia_length}"/>
+        </geometry>
+      </collision>
     </link>
     <joint name="${leg_name}_tibia_joint" type="revolute">
+      <origin xyz="${femur_length} 0 0" rpy="0 0 0"/>
       <parent link="${leg_name}_femur_link"/>
       <child link="${leg_name}_tibia_link"/>
-      <origin xyz="0 0 ${-femur_length}" rpy="0 0 0"/>
       <axis xyz="0 1 0"/>
-      <limit lower="${joint_lower_limit}" upper="${joint_upper_limit}" effort="10" velocity="1.0"/>
+      <limit lower="${joint_lower_limit}" upper="${joint_upper_limit}" effort="10" velocity="4"/>
+    </joint>
+    <!-- Foot with Contact Sensor -->
+    <link name="${leg_name}_foot">
+      <inertial>
+        <mass value="0.01"/>
+        <inertia ixx="1e-6" ixy="0" ixz="0" iyy="1e-6" iyz="0" izz="1e-6"/>
+      </inertial>
+      <visual>
+        <origin xyz="0 0 0" rpy="0 0 0"/>
+        <geometry>
+          <sphere radius="0.02"/>
+        </geometry>
+        <material name="black">
+          <color rgba="0.1 0.1 0.1 1.0"/>
+        </material>
+      </visual>
+      <collision name="${leg_name}_foot_collision">
+        <origin xyz="0 0 0" rpy="0 0 0"/>
+        <geometry>
+          <sphere radius="0.02"/>
+        </geometry>
+        <surface>
+          <friction>
+            <ode>
+              <mu>1.0</mu>
+              <mu2>1.0</mu2>
+            </ode>
+          </friction>
+        </surface>
+      </collision>
+    </link>
+    <joint name="${leg_name}_foot_joint" type="fixed">
+      <origin xyz="${tibia_length} 0 0" rpy="0 0 0"/>
+      <parent link="${leg_name}_tibia_link"/>
+      <child link="${leg_name}_foot"/>
     </joint>
   </xacro:macro>
-  <!-- CREATE 6 LEGS -->
-  <xacro:leg leg_name="leg_1" hx="${base_radius*0.866}" hy="${base_radius*0.5}" hz="${base_height}" hr="0" hp="0" hyaw="0.524"/>
-  <xacro:leg leg_name="leg_2" hx="0" hy="${base_radius}" hz="${base_height}" hr="0" hp="0" hyaw="1.571"/>
-  <xacro:leg leg_name="leg_3" hx="${-base_radius*0.866}" hy="${base_radius*0.5}" hz="${base_height}" hr="0" hp="0" hyaw="2.618"/>
-  <xacro:leg leg_name="leg_4" hx="${-base_radius*0.866}" hy="${-base_radius*0.5}" hz="${base_height}" hr="0" hp="0" hyaw="3.665"/>
-  <xacro:leg leg_name="leg_5" hx="0" hy="${-base_radius}" hz="${base_height}" hr="0" hp="0" hyaw="4.712"/>
-  <xacro:leg leg_name="leg_6" hx="${base_radius*0.866}" hy="${-base_radius*0.5}" hz="${base_height}" hr="0" hp="0" hyaw="5.759"/>
-  <!-- ROS2 CONTROL - GAZEBO HARDWARE INTERFACE -->
+  <!-- CREATE 6 LEGS (60 degrees apart) -->
+  <xacro:leg leg_name="leg_1" hx="${base_radius}" hy="0.0" angle="0"/>
+  <xacro:leg leg_name="leg_2" hx="${base_radius*0.5}" hy="${base_radius*0.866}" angle="1.0472"/>
+  <xacro:leg leg_name="leg_3" hx="${-base_radius*0.5}" hy="${base_radius*0.866}" angle="2.0944"/>
+  <xacro:leg leg_name="leg_4" hx="${-base_radius}" hy="0.0" angle="3.14159"/>
+  <xacro:leg leg_name="leg_5" hx="${-base_radius*0.5}" hy="${-base_radius*0.866}" angle="-2.0944"/>
+  <xacro:leg leg_name="leg_6" hx="${base_radius*0.5}" hy="${-base_radius*0.866}" angle="-1.0472"/>
+  <!-- ROS2 CONTROL -->
   <ros2_control name="HexapodSystem" type="system">
     <hardware>
       <plugin>gz_ros2_control/GazeboSimSystem</plugin>
+      <param name="example_param_hw_start_duration_sec">0.0</param>
+      <param name="example_param_hw_stop_duration_sec">0.0</param>
+      <param name="example_param_hw_slowdown">1.0</param>
     </hardware>
-    <!-- DEFINE ALL JOINTS -->
-    <xacro:macro name="joint_interface" params="joint_name">
-      <joint name="${joint_name}">
-        <command_interface name="position">
-          <param name="min">${joint_lower_limit}</param>
-          <param name="max">${joint_upper_limit}</param>
-        </command_interface>
+    <xacro:macro name="joint_control" params="leg_name">
+      <joint name="${leg_name}_hip_joint">
+        <command_interface name="position"/>
+        <state_interface name="position"/>
+        <state_interface name="velocity"/>
+      </joint>
+      <joint name="${leg_name}_femur_joint">
+        <command_interface name="position"/>
+        <state_interface name="position"/>
+        <state_interface name="velocity"/>
+      </joint>
+      <joint name="${leg_name}_tibia_joint">
+        <command_interface name="position"/>
         <state_interface name="position"/>
         <state_interface name="velocity"/>
       </joint>
     </xacro:macro>
-    <xacro:joint_interface joint_name="leg_1_hip_joint"/>
-    <xacro:joint_interface joint_name="leg_1_femur_joint"/>
-    <xacro:joint_interface joint_name="leg_1_tibia_joint"/>
-    <xacro:joint_interface joint_name="leg_2_hip_joint"/>
-    <xacro:joint_interface joint_name="leg_2_femur_joint"/>
-    <xacro:joint_interface joint_name="leg_2_tibia_joint"/>
-    <xacro:joint_interface joint_name="leg_3_hip_joint"/>
-    <xacro:joint_interface joint_name="leg_3_femur_joint"/>
-    <xacro:joint_interface joint_name="leg_3_tibia_joint"/>
-    <xacro:joint_interface joint_name="leg_4_hip_joint"/>
-    <xacro:joint_interface joint_name="leg_4_femur_joint"/>
-    <xacro:joint_interface joint_name="leg_4_tibia_joint"/>
-    <xacro:joint_interface joint_name="leg_5_hip_joint"/>
-    <xacro:joint_interface joint_name="leg_5_femur_joint"/>
-    <xacro:joint_interface joint_name="leg_5_tibia_joint"/>
-    <xacro:joint_interface joint_name="leg_6_hip_joint"/>
-    <xacro:joint_interface joint_name="leg_6_femur_joint"/>
-    <xacro:joint_interface joint_name="leg_6_tibia_joint"/>
+    <xacro:joint_control leg_name="leg_1"/>
+    <xacro:joint_control leg_name="leg_2"/>
+    <xacro:joint_control leg_name="leg_3"/>
+    <xacro:joint_control leg_name="leg_4"/>
+    <xacro:joint_control leg_name="leg_5"/>
+    <xacro:joint_control leg_name="leg_6"/>
   </ros2_control>
   <!-- GAZEBO ROS2 CONTROL PLUGIN -->
@@ -187,3 +244,39 @@
     </plugin>
   </gazebo>
+  <!-- GAZEBO SENSOR PLUGINS -->
+  <gazebo reference="imu_link">
+    <sensor name="imu_sensor" type="imu">
+      <always_on>true</always_on>
+      <update_rate>50</update_rate>
+      <visualize>true</visualize>
+      <topic>imu/data</topic>
+    </sensor>
+  </gazebo>
+  <gazebo reference="lidar_link">
+    <sensor name="lidar_sensor" type="gpu_lidar">
+      <update_rate>10</update_rate>
+      <topic>scan</topic>
+      <ray>
+        <scan>
+          <horizontal>
+            <samples>360</samples>
+            <resolution>1</resolution>
+            <min_angle>-3.14159</min_angle>
+            <max_angle>3.14159</max_angle>
+          </horizontal>
+        </scan>
+        <range>
+          <min>0.12</min>
+          <max>10.0</max>
+          <resolution>0.01</resolution>
+        </range>
+      </ray>
+    </sensor>
+  </gazebo>
+  <gazebo reference="imu_joint">
+    <preserveFixedJoint>true</preserveFixedJoint>
+  </gazebo>
+  <gazebo reference="lidar_joint">
+    <preserveFixedJoint>true</preserveFixedJoint>
+  </gazebo>
 </robot>

Commit message: sensors goddamn workgit add *git add *!

File: src/hexapod_ws/description/hexapod.urdf.xacro (robot description, xacro)
@@ -206,11 +206,7 @@
   <xacro:leg leg_name="leg_5" hx="${-base_radius*0.5}" hy="${-base_radius*0.866}" angle="-2.0944"/>
   <xacro:leg leg_name="leg_6" hx="${base_radius*0.5}" hy="${-base_radius*0.866}" angle="-1.0472"/>
-  <!-- ROS2 CONTROL -->
   <ros2_control name="HexapodSystem" type="system">
     <hardware>
       <plugin>gz_ros2_control/GazeboSimSystem</plugin>
-      <param name="example_param_hw_start_duration_sec">0.0</param>
-      <param name="example_param_hw_stop_duration_sec">0.0</param>
-      <param name="example_param_hw_slowdown">1.0</param>
     </hardware>
     <xacro:macro name="joint_control" params="leg_name">
@@ -238,24 +234,31 @@
     <xacro:joint_control leg_name="leg_6"/>
   </ros2_control>
-  <!-- GAZEBO ROS2 CONTROL PLUGIN -->
   <gazebo>
-    <plugin filename="libgz_ros2_control-system.so" name="gz_ros2_control::GazeboSimROS2ControlPlugin">
+    <plugin filename="gz-sim-joint-state-publisher-system" name="gz::sim::systems::JointStatePublisher">
+      <topic>joint_states</topic>
+    </plugin>
+    <plugin filename="gz_ros2_control-system" name="gz_ros2_control::GazeboSimROS2ControlPlugin">
       <parameters>$(find hexapod_ws)/config/parameters.yaml</parameters>
     </plugin>
   </gazebo>
-  <!-- GAZEBO SENSOR PLUGINS -->
+  <gazebo reference="imu_joint"><preserveFixedJoint>true</preserveFixedJoint></gazebo>
+  <gazebo reference="lidar_joint"><preserveFixedJoint>true</preserveFixedJoint></gazebo>
   <gazebo reference="imu_link">
     <sensor name="imu_sensor" type="imu">
       <always_on>true</always_on>
-      <update_rate>50</update_rate>
+      <update_rate>100</update_rate>
       <visualize>true</visualize>
-      <topic>imu/data</topic>
-    </sensor>
+      <topic>imu</topic>
+      <gz_frame_id>imu_link</gz_frame_id>
+      <imu/> </sensor>
   </gazebo>
   <gazebo reference="lidar_link">
-    <sensor name="lidar_sensor" type="gpu_lidar">
+    <sensor name="gpu_lidar" type="gpu_lidar">
+      <always_on>true</always_on>
       <update_rate>10</update_rate>
+      <visualize>true</visualize>
       <topic>scan</topic>
-      <ray>
+      <gz_frame_id>lidar_link</gz_frame_id>
+      <lidar>
         <scan>
           <horizontal>
@@ -271,12 +274,21 @@
           <resolution>0.01</resolution>
         </range>
-      </ray>
+      </lidar>
     </sensor>
   </gazebo>
-  <gazebo reference="imu_joint">
-    <preserveFixedJoint>true</preserveFixedJoint>
-  </gazebo>
-  <gazebo reference="lidar_joint">
-    <preserveFixedJoint>true</preserveFixedJoint>
-  </gazebo>
+  <xacro:macro name="foot_sensor" params="num">
+    <gazebo reference="leg_${num}_foot">
+      <sensor name="leg_${num}_contact" type="contact">
+        <always_on>true</always_on>
+        <update_rate>50</update_rate>
+        <topic>leg_${num}_contact</topic>
+        <gz_frame_id>leg_${num}_foot</gz_frame_id>
+        <contact>
+          <collision>leg_${num}_foot_collision</collision>
+        </contact>
+      </sensor>
+    </gazebo>
+  </xacro:macro>
+  <xacro:foot_sensor num="1"/><xacro:foot_sensor num="2"/><xacro:foot_sensor num="3"/>
+  <xacro:foot_sensor num="4"/><xacro:foot_sensor num="5"/><xacro:foot_sensor num="6"/>
 </robot>
