Commit message: >made changes to movement >added force sensors to allow hexapod to know if its touching the ground or not >minor movement glitches fixed

File: src/hexapod_ws/description/hexapod.urdf.xacro (robot description, xacro)
@@ -73,5 +73,4 @@
   <!-- LEG MACRO -->
   <xacro:macro name="leg" params="leg_name hx hy angle">
-    <!-- Hip Link (Coxa) -->
     <link name="${leg_name}_hip_link">
       <inertial>
@@ -82,16 +81,10 @@
       <visual>
         <origin xyz="${hip_length/2} 0 0" rpy="0 1.5708 0"/>
-        <geometry>
-          <cylinder radius="${leg_radius}" length="${hip_length}"/>
-        </geometry>
-        <material name="black">
-          <color rgba="0.1 0.1 0.1 1.0"/>
-        </material>
+        <geometry><cylinder radius="${leg_radius}" length="${hip_length}"/></geometry>
+        <material name="black"><color rgba="0.1 0.1 0.1 1.0"/></material>
       </visual>
       <collision>
         <origin xyz="${hip_length/2} 0 0" rpy="0 1.5708 0"/>
-        <geometry>
-          <cylinder radius="${leg_radius}" length="${hip_length}"/>
-        </geometry>
+        <geometry><cylinder radius="${leg_radius}" length="${hip_length}"/></geometry>
       </collision>
     </link>
@@ -103,5 +96,4 @@
       <limit lower="${joint_lower_limit}" upper="${joint_upper_limit}" effort="10" velocity="4"/>
     </joint>
-    <!-- Femur Link -->
     <link name="${leg_name}_femur_link">
       <inertial>
@@ -112,16 +104,10 @@
       <visual>
         <origin xyz="${femur_length/2} 0 0" rpy="0 1.5708 0"/>
-        <geometry>
-          <cylinder radius="${leg_radius}" length="${femur_length}"/>
-        </geometry>
-        <material name="red">
-          <color rgba="0.8 0.2 0.2 1.0"/>
-        </material>
+        <geometry><cylinder radius="${leg_radius}" length="${femur_length}"/></geometry>
+        <material name="red"><color rgba="0.8 0.2 0.2 1.0"/></material>
       </visual>
       <collision>
         <origin xyz="${femur_length/2} 0 0" rpy="0 1.5708 0"/>
-        <geometry>
-          <cylinder radius="${leg_radius}" length="${femur_length}"/>
-        </geometry>
+        <geometry><cylinder radius="${leg_radius}" length="${femur_length}"/></geometry>
       </collision>
     </link>
@@ -133,5 +119,4 @@
       <limit lower="${joint_lower_limit}" upper="${joint_upper_limit}" effort="10" velocity="4"/>
     </joint>
-    <!-- Tibia Link -->
     <link name="${leg_name}_tibia_link">
       <inertial>
@@ -142,16 +127,10 @@
       <visual>
         <origin xyz="${tibia_length/2} 0 0" rpy="0 1.5708 0"/>
-        <geometry>
-          <cylinder radius="${leg_radius}" length="${tibia_length}"/>
-        </geometry>
-        <material name="blue">
-          <color rgba="0.2 0.2 0.8 1.0"/>
-        </material>
+        <geometry><cylinder radius="${leg_radius}" length="${tibia_length}"/></geometry>
+        <material name="blue"><color rgba="0.2 0.2 0.8 1.0"/></material>
       </visual>
       <collision>
         <origin xyz="${tibia_length/2} 0 0" rpy="0 1.5708 0"/>
-        <geometry>
-          <cylinder radius="${leg_radius}" length="${tibia_length}"/>
-        </geometry>
+        <geometry><cylinder radius="${leg_radius}" length="${tibia_length}"/></geometry>
       </collision>
     </link>
@@ -163,5 +142,4 @@
       <limit lower="${joint_lower_limit}" upper="${joint_upper_limit}" effort="10" velocity="4"/>
     </joint>
-    <!-- Foot with Contact Sensor -->
     <link name="${leg_name}_foot">
       <inertial>
@@ -171,21 +149,14 @@
       <visual>
         <origin xyz="0 0 0" rpy="0 0 0"/>
-        <geometry>
-          <sphere radius="0.02"/>
-        </geometry>
-        <material name="black">
-          <color rgba="0.1 0.1 0.1 1.0"/>
-        </material>
+        <geometry><sphere radius="0.02"/></geometry>
+        <material name="black"><color rgba="0.1 0.1 0.1 1.0"/></material>
       </visual>
       <collision name="${leg_name}_foot_collision">
         <origin xyz="0 0 0" rpy="0 0 0"/>
-        <geometry>
-          <sphere radius="0.02"/>
-        </geometry>
+        <geometry><sphere radius="0.02"/></geometry>
         <surface>
           <friction>
             <ode>
-              <mu>1.0</mu>
-              <mu2>1.0</mu2>
+              <mu>1.0</mu> <mu2>1.0</mu2>
             </ode>
           </friction>
@@ -193,8 +164,10 @@
       </collision>
     </link>
-    <joint name="${leg_name}_foot_joint" type="fixed">
+    <joint name="${leg_name}_foot_joint" type="prismatic">
       <origin xyz="${tibia_length} 0 0" rpy="0 0 0"/>
       <parent link="${leg_name}_tibia_link"/>
       <child link="${leg_name}_foot"/>
+      <axis xyz="1 0 0"/> <limit lower="-0.05" upper="0.0" effort="100" velocity="10"/>
+      <dynamics damping="1.0" friction="0" spring_stiffness="1" spring_reference="0.0"/>
     </joint>
   </xacro:macro>
@@ -215,4 +188,5 @@
         <state_interface name="position"/>
         <state_interface name="velocity"/>
+        <state_interface name="effort"/>
       </joint>
       <joint name="${leg_name}_femur_joint">
@@ -220,4 +194,5 @@
         <state_interface name="position"/>
         <state_interface name="velocity"/>
+        <state_interface name="effort"/>
       </joint>
       <joint name="${leg_name}_tibia_joint">
@@ -225,4 +200,8 @@
         <state_interface name="position"/>
         <state_interface name="velocity"/>
+        <state_interface name="effort"/>
+      </joint>
+      <joint name="${leg_name}_foot_joint">
+        <state_interface name="position"/> <state_interface name="velocity"/>
       </joint>
     </xacro:macro>
@@ -235,7 +214,4 @@
   </ros2_control>
   <gazebo>
-    <plugin filename="gz-sim-joint-state-publisher-system" name="gz::sim::systems::JointStatePublisher">
-      <topic>joint_states</topic>
-    </plugin>
     <plugin filename="gz_ros2_control-system" name="gz_ros2_control::GazeboSimROS2ControlPlugin">
       <parameters>$(find hexapod_ws)/config/parameters.yaml</parameters>
@@ -277,18 +253,3 @@
     </sensor>
   </gazebo>
-  <xacro:macro name="foot_sensor" params="num">
-    <gazebo reference="leg_${num}_foot">
-      <sensor name="leg_${num}_contact" type="contact">
-        <always_on>true</always_on>
-        <update_rate>50</update_rate>
-        <topic>leg_${num}_contact</topic>
-        <gz_frame_id>leg_${num}_foot</gz_frame_id>
-        <contact>
-          <collision>leg_${num}_foot_collision</collision>
-        </contact>
-      </sensor>
-    </gazebo>
-  </xacro:macro>
-  <xacro:foot_sensor num="1"/><xacro:foot_sensor num="2"/><xacro:foot_sensor num="3"/>
-  <xacro:foot_sensor num="4"/><xacro:foot_sensor num="5"/><xacro:foot_sensor num="6"/>
 </robot>
